File: N64DEV.sch (KiCad schematic (older format))
At the start: 0 parts

Commit message: Add reference
Changed lines of the file:
@@
 $Descr A4 11693 8268
 encoding utf-8
-Sheet 1 7
+Sheet 1 8
 Title "Rare N64DEV V3 - Overview"
 Date "2021-12-30"
@@
 Comment4 ""
 $EndDescr
-$Sheet
-S 4000 1050 2500 1050
-U 61D8F000
-F0 "TopN64Bus" 50
-F1 "TopN64Bus.sch" 50
-$EndSheet
 $Sheet
 S 4000 2350 2500 850
@@
 $EndSheet
 $Sheet
-S 2700 1050 1150 5600
-U 61D8F1A6
-F0 "DRAM" 50
-F1 "DRAM.sch" 50
-$EndSheet
-$Sheet
 S 4000 5750 2500 950
 U 61D8F286
@@
 F1 "BottomN64Bus.sch" 50
 $EndSheet
+$Sheet
+S 2600 850  1100 5650
+U 62445696
+F0 "DRAM_Back" 50
+F1 "DRAM_Back.sch" 50
+$EndSheet
+$Sheet
+S 4000 1050 2500 1050
+U 61D8F000
+F0 "TopN64Bus" 50
+F1 "TopN64Bus.sch" 50
+$EndSheet
+$Sheet
+S 2700 1050 1150 5600
+U 61D8F1A6
+F0 "DRAM_Front" 50
+F1 "DRAM_Front.sch" 50
+$EndSheet
 $EndSCHEMATC
