File: SCSI.sch (KiCad schematic (older format))
At the start: 4 parts

Commit message: Add reference
Parts:
- P1: renamed from J?; value Conn_02x34_SCSI-III -> SCSI_HD68
- gave numbers to parts that had none: 3
Connections:
- wire segments 0 -> 176
Other:
- moved on the sheet: U1, U31, U4
