File: TopN64Bus.sch (KiCad schematic (older format))
At the start: 2 parts

Commit message: Add reference
Parts:
- CON1: renamed from J?; value Conn_02x25_N64_Cartridge -> N64_Cartridge_Slot
- gave numbers to parts that had none: 1
Connections:
- wire segments 0 -> 59
Other:
- moved on the sheet: CON1, P5
Changed lines of the file:
@@
 $Descr A4 11693 8268
 encoding utf-8
-Sheet 2 7
+Sheet 7 8
 Title "Rare N64DEV V3 - Top N64 Bus"
 Date "2021-12-30"
@@
 $EndDescr
 $Comp
-L N64DEV:Conn_02x25_N64_Cartridge J?
+L N64DEV:Conn_02x25_N64_Cartridge CON1
 U 1 1 61E1FE33
-P 8400 3250
-F 0 "J?" H 8450 4667 50  0000 C CNN
-F 1 "Conn_02x25_N64_Cartridge" H 8450 4576 50  0000 C CNN
-F 2 "" H 8400 3250 50  0001 C CNN
-F 3 "~" H 8400 3250 50  0001 C CNN
-	1    8400 3250
+P 3950 3350
+F 0 "CON1" H 4000 4767 50  0000 C CNN
+F 1 "N64_Cartridge_Slot" H 4000 4676 50  0000 C CNN
+F 2 "" H 3950 3350 50  0001 C CNN
+F 3 "~" H 3950 3350 50  0001 C CNN
+	1    3950 3350
 	1    0    0    -1
 $EndComp
 $Comp
-L N64DEV:DB9_Female J?
+L N64DEV:DB9_Female P5
 U 1 1 61E22446
-P 4550 1800
-F 0 "J?" H 4730 1846 50  0000 L CNN
-F 1 "DB9_Female" H 4730 1755 50  0000 L CNN
-F 2 "" H 4550 1800 50  0001 C CNN
-F 3 " ~" H 4550 1800 50  0001 C CNN
-	1    4550 1800
+P 8800 3250
+F 0 "P5" H 8980 3296 50  0000 L CNN
+F 1 "DB9_Female" H 8980 3205 50  0000 L CNN
+F 2 "" H 8800 3250 50  0001 C CNN
+F 3 " ~" H 8800 3250 50  0001 C CNN
+	1    8800 3250
 	1    0    0    -1
 $EndComp
+Wire Wire Line
+	3750 2550 3500 2550
+Wire Wire Line
+	3750 2450 3500 2450
+Wire Wire Line
+	3750 2350 3500 2350
+Wire Wire Line
+	3750 2250 3500 2250
+Wire Wire Line
+	3750 2150 3500 2150
+Wire Wire Line
+	3750 3050 3500 3050
+Wire Wire Line
+	3750 2950 3500 2950
+Wire Wire Line
+	3750 2850 3500 2850
+Wire Wire Line
+	3750 2750 3500 2750
+Wire Wire Line
+	3750 2650 3500 2650
+Wire Wire Line
+	3750 3550 3500 3550
+Wire Wire Line
+	3750 3450 3500 3450
+Wire Wire Line
+	3750 3350 3500 3350
+Wire Wire Line
+	3750 3250 3500 3250
+Wire Wire Line
+	3750 3150 3500 3150
+Wire Wire Line
+	3750 4050 3500 4050
+Wire Wire Line
+	3750 3950 3500 3950
+Wire Wire Line
+	3750 3850 3500 3850
+Wire Wire Line
+	3750 3750 3500 3750
+Wire Wire Line
+	3750 3650 3500 3650
+Wire Wire Line
+	3750 4550 3500 4550
+Wire Wire Line
+	3750 4450 3500 4450
+Wire Wire Line
+	3750 4350 3500 4350
+Wire Wire Line
+	3750 4250 3500 4250
+Wire Wire Line
+	3750 4150 3500 4150
+Wire Wire Line
+	4250 4150 4500 4150
+Wire Wire Line
+	4250 4250 4500 4250
+Wire Wire Line
+	4250 4350 4500 4350
+Wire Wire Line
+	4250 4450 4500 4450
+Wire Wire Line
+	4250 4550 4500 4550
+Wire Wire Line
+	4250 3650 4500 3650
+Wire Wire Line
+	4250 3750 4500 3750
+Wire Wire Line
+	4250 3850 4500 3850
+Wire Wire Line
+	4250 3950 4500 3950
+Wire Wire Line
+	4250 4050 4500 4050
+Wire Wire Line
+	4250 3150 4500 3150
+Wire Wire Line
+	4250 3250 4500 3250
+Wire Wire Line
+	4250 3350 4500 3350
+Wire Wire Line
+	4250 3450 4500 3450
+Wire Wire Line
+	4250 3550 4500 3550
+Wire Wire Line
+	4250 2650 4500 2650
+Wire Wire Line
+	4250 2750 4500 2750
+Wire Wire Line
+	4250 2850 4500 2850
+Wire Wire Line
+	4250 2950 4500 2950
+Wire Wire Line
+	4250 3050 4500 3050
+Wire Wire Line
+	4250 2150 4500 2150
+Wire Wire Line
+	4250 2250 4500 2250
+Wire Wire Line
+	4250 2350 4500 2350
+Wire Wire Line
+	4250 2450 4500 2450
+Wire Wire Line
+	4250 2550 4500 2550
+Wire Wire Line
+	8500 3250 8250 3250
+Wire Wire Line
+	8500 3150 8250 3150
+Wire Wire Line
+	8500 3050 8250 3050
+Wire Wire Line
+	8500 2950 8250 2950
+Wire Wire Line
+	8500 2850 8250 2850
+Wire Wire Line
+	8500 3650 8250 3650
+Wire Wire Line
+	8500 3550 8250 3550
+Wire Wire Line
+	8500 3450 8250 3450
+Wire Wire Line
+	8500 3350 8250 3350
 $EndSCHEMATC

Commit message: MCU start
Connections:
- net labels added: +12V, +3V3, GND, N64_AD0, N64_AD1, N64_AD10, N64_AD11, N64_AD12, N64_AD13, N64_AD14, N64_AD15, N64_AD2, N64_AD3, N64_AD4, N64_AD5, N64_AD6, N64_AD7, N64_AD8, N64_AD9, N64_ALE_H, N64_ALE_L, N64_CIC_DI, N64_CIC_DO, N64_PIF_CLK, N64_~RESET~, N64_~W~
- wire segments 59 -> 65
- no-connect marks 0 -> 13
Other:
- note added: "Cartridge label facing up (unlike Partner)"
- note added: "Only wired for SRAM & Flash save"

Commit message: MCU WIP
Connections:
- net labels added: N64_TOP_~R~
- wire segments 65 -> 66
- no-connect marks 13 -> 12
Changed lines of the file:
@@
 P 4100 4500
 AR Path="/61D8F286/628D6B5B" Ref="#PWR?"  Part="1"
-AR Path="/61D8F000/628D6B5B" Ref="#PWR?"  Part="1"
-F 0 "#PWR?" H 4100 4250 50  0001 C CNN
+AR Path="/61D8F000/628D6B5B" Ref="#PWR0169"  Part="1"
+F 0 "#PWR0169" H 4100 4250 50  0001 C CNN
 F 1 "GND" H 4105 4327 50  0000 C CNN
 F 2 "" H 4100 4500 50  0001 C CNN
@@
 P 4700 4500
 AR Path="/61D8F286/628D6B62" Ref="#PWR?"  Part="1"
-AR Path="/61D8F000/628D6B62" Ref="#PWR?"  Part="1"
-F 0 "#PWR?" H 4700 4250 50  0001 C CNN
+AR Path="/61D8F000/628D6B62" Ref="#PWR0170"  Part="1"
+F 0 "#PWR0170" H 4700 4250 50  0001 C CNN
 F 1 "GND" H 4705 4327 50  0000 C CNN
 F 2 "" H 4700 4500 50  0001 C CNN
@@
 P 4000 1750
 AR Path="/61D8F286/628D6B6D" Ref="#PWR?"  Part="1"
-AR Path="/61D8F000/628D6B6D" Ref="#PWR?"  Part="1"
-F 0 "#PWR?" H 4000 1600 50  0001 C CNN
+AR Path="/61D8F000/628D6B6D" Ref="#PWR0171"  Part="1"
+F 0 "#PWR0171" H 4000 1600 50  0001 C CNN
 F 1 "+3V3" H 4015 1923 50  0000 C CNN
 F 2 "" H 4000 1750 50  0001 C CNN
@@
 P 4800 1750
 AR Path="/61D8F286/628D6B75" Ref="#PWR?"  Part="1"
-AR Path="/61D8F000/628D6B75" Ref="#PWR?"  Part="1"
-F 0 "#PWR?" H 4800 1600 50  0001 C CNN
+AR Path="/61D8F000/628D6B75" Ref="#PWR0172"  Part="1"
+F 0 "#PWR0172" H 4800 1600 50  0001 C CNN
 F 1 "+3V3" H 4815 1923 50  0000 C CNN
 F 2 "" H 4800 1750 50  0001 C CNN
@@
 P 4900 1900
 AR Path="/61D8F286/628D6BC7" Ref="#PWR?"  Part="1"
-AR Path="/61D8F000/628D6BC7" Ref="#PWR?"  Part="1"
-F 0 "#PWR?" H 4900 1750 50  0001 C CNN
+AR Path="/61D8F000/628D6BC7" Ref="#PWR0173"  Part="1"
+F 0 "#PWR0173" H 4900 1750 50  0001 C CNN
 F 1 "+12V" H 4915 2073 50  0000 C CNN
 F 2 "" H 4900 1900 50  0001 C CNN
@@
 P 3900 1900
 AR Path="/61D8F286/628D6BCE" Ref="#PWR?"  Part="1"
-AR Path="/61D8F000/628D6BCE" Ref="#PWR?"  Part="1"
-F 0 "#PWR?" H 3900 1750 50  0001 C CNN
+AR Path="/61D8F000/628D6BCE" Ref="#PWR0174"  Part="1"
+F 0 "#PWR0174" H 3900 1750 50  0001 C CNN
 F 1 "+12V" H 3850 2100 50  0000 C CNN
 F 2 "" H 3900 1900 50  0001 C CNN
@@
 Wire Wire Line
 	3900 3100 3900 1900
-NoConn ~ 4150 2800
 Wire Wire Line
 	3000 2600 4150 2600
@@
 P 8500 3850
 AR Path="/61D8F286/62926AC4" Ref="#PWR?"  Part="1"
-AR Path="/61D8F000/62926AC4" Ref="#PWR?"  Part="1"
-F 0 "#PWR?" H 8500 3600 50  0001 C CNN
+AR Path="/61D8F000/62926AC4" Ref="#PWR0175"  Part="1"
+F 0 "#PWR0175" H 8500 3600 50  0001 C CNN
 F 1 "GND" H 8505 3677 50  0000 C CNN
 F 2 "" H 8500 3850 50  0001 C CNN
@@
 P 8500 2700
 AR Path="/61D8F286/62928B9C" Ref="#PWR?"  Part="1"
-AR Path="/61D8F000/62928B9C" Ref="#PWR?"  Part="1"
-F 0 "#PWR?" H 8500 2550 50  0001 C CNN
+AR Path="/61D8F000/62928B9C" Ref="#PWR0176"  Part="1"
+F 0 "#PWR0176" H 8500 2550 50  0001 C CNN
 F 1 "+3V3" H 8515 2873 50  0000 C CNN
 F 2 "" H 8500 2700 50  0001 C CNN
@@
 Text Label 8250 3250 2    50   ~ 0
 N64_~RESET~
+Wire Wire Line
+	4150 2800 3000 2800
+Text Label 3000 2800 0    50   ~ 0
+N64_TOP_~R~
 $EndSCHEMATC
