File: FPGA.sch (KiCad schematic (older format))
At the start: 7 parts

Commit message: Add reference
Parts:
- P3: renamed from J?; value Conn_02x05_Odd_Even -> FPGA_JTAG
- gave numbers to parts that had none: 2
Connections:
- wire segments 0 -> 218
Other:
- moved on the sheet: P3, U18A, U18B, U18C, U18D, U18E, U20

Commit message: MCU start
Parts:
- added C47, C48, C52, C55, C56, C57, C60, C66, C67, C70: ~, symbol N64DEV:C_Small
- added C72: ~, symbol N64DEV:CP_Small
- added R25, R26: 27, symbol N64DEV:R_Small_US
- added R27, R32, R33, R34, R35, R37: 1K, symbol N64DEV:R_Small_US
- added R38: 4K7, symbol N64DEV:R_Small_US
- added RP2, RP3, RP5, RP7: QSP16J-1-220, Package_SO:SSOP-16_3.9x4.9mm_P0.635mm, symbol N64DEV:QSP16J
Connections:
- net labels added: +3V3, +5V, DRAM_~UCAS~_~LCAS~, DRAM_~W~, GND, MCU_A21, N64_AD0, N64_AD1, N64_AD10, N64_AD11, N64_AD12, N64_AD13, N64_AD14, N64_AD15, N64_AD2, N64_AD3, N64_AD4, N64_AD5, N64_AD6, N64_AD7, N64_AD8, N64_AD9, N64_ALE_H, N64_ALE_L, N64_LA_INT4, N64_NMI, N64_RA_PIF_EN, N64_VC_WRST, N64_~R~, N64_~W~
- wire segments 218 -> 244
- no-connect marks 0 -> 4
Other:
- moved on the sheet: P3, U18A, U18D, U18E, U20

Commit message: MCU WIP
Parts:
- added C71: 10u, symbol N64DEV:CP1_Small
- renumbered R38 to R36
Connections:
- net labels added: N64_TOP_~R~
- wire segments 244 -> 248

Commit message: Latest
Connections:
- net labels added: MCU_CLK_OUT
Changed lines of the file:
@@
 Wire Wire Line
 	7450 3150 8300 3150
+Text Label 6500 5750 0    50   ~ 0
+MCU_CLK_OUT
 $EndSCHEMATC
