File: MCU.sch (KiCad schematic (older format))
At the start: 8 parts

Commit message: Add reference
Parts:
- P2: renamed from J?; value Conn_02x05_Odd_Even -> MCU_JTAG
- gave numbers to parts that had none: 7
Connections:
- wire segments 0 -> 313
Other:
- moved on the sheet: P2, U15, U16

Commit message: MCU start
Parts:
- added R12, R15, R5, R6, R9: 4K7, symbol N64DEV:R_Small_US
Connections:
- net labels added: +5V, MCU_A21
- wire segments 313 -> 322
Other:
- moved on the sheet: P2, U12, U13, U15, U16

Commit message: MCU WIP
Parts:
- added C31, C33: ~, symbol N64DEV:C_Small
- added R10, R11, R13, R16, R17, R?: 4K7, symbol N64DEV:R_Small_US
- added R7: 10M, symbol N64DEV:R_Small_US
- added R8: 470, symbol N64DEV:R_Small_US
- added X2: 3.6864, symbol N64DEV:Crystal_Small
Connections:
- net labels added: GND, MCU_A0, MCU_A1, MCU_A10, MCU_A11, MCU_A12, MCU_A13, MCU_A14, MCU_A15, MCU_A16, MCU_A17, MCU_A18, MCU_A19, MCU_A2, MCU_A20, MCU_A22, MCU_A23, MCU_A3, MCU_A4, MCU_A5, MCU_A6, MCU_A7, MCU_A8, MCU_A9, MCU_D0, MCU_D1, MCU_D10, MCU_D11, MCU_D12, MCU_D13, MCU_D14, MCU_D15, MCU_D2, MCU_D3, MCU_D4, MCU_D5, MCU_D6, MCU_D7, MCU_D8, MCU_D9
- wire segments 322 -> 339
Other:
- moved on the sheet: R12, R15, R5, R6, R9, U13, U15, U8, U9

Commit message: Latest
Parts:
- added C+, C-, C38, C39, C40: ~, symbol N64DEV:C_Small
- added R20: 4K7, symbol N64DEV:R_Small_US
- added R21: 1K, symbol N64DEV:R_Small_US
- added R?: 10M, symbol N64DEV:R_Small_US
- added R?: 330K, symbol N64DEV:R_Small_US
- added RP1: 9X-1-472, Resistor_THT:R_Array_SIP9, symbol N64DEV:R_Network08_US
- added S1: Conn_01x02, symbol N64DEV:Conn_01x02
- added X3: 3.6864, symbol N64DEV:Crystal_Small
Connections:
- net labels added: MCU_CLKOUT, MCU_FREEZE, MCU_~AS~, MCU_~BERR~, MCU_~BGACK~, MCU_~BKPT~, MCU_~BR~, MCU_~DSACK1~, MCU_~DS~, MCU_~HALT~, MCU_~IFETCH~, MCU_~IPIPE~, MCU_~RESET~
- wire segments 339 -> 373
Other:
- moved on the sheet: P2, R10, R12, R13, R15, R5, R6, R9, U12, U15
